Commit message: feat: repair controller association
Issue: target position for trajectory sampler

File: kuka_arm/urdf/iiwa14.xacro (robot description, xacro)
@@ -27,8 +27,13 @@
     </joint>
     <link name="base_link">
-      <inertial>
+      <!--<inertial>
         <origin xyz="-0.1 0 0.07" rpy="0 0 0"/>
         <mass value="5"/>
         <inertia ixx="0.05"  ixy="0"  ixz="0" iyy="0.06" iyz="0" izz="0.03" />
+      </inertial>-->
+      <inertial>
+        <origin xyz="-0.1 0 0.07" rpy="0 0 0"/>
+        <mass value="50"/>
+        <inertia ixx="0.5"  ixy="0"  ixz="0" iyy="0.6" iyz="0" izz="0.3" />
       </inertial>
       <visual>

File: kuka_arm/urdf/target.urdf.xacro (robot description, xacro)
@@ -10,5 +10,5 @@
       <origin xyz="0 0 0"/>
       <geometry>
-        <cylinder radius="0.01" length="0.08"/>
+        <cylinder radius="0.02" length="0.08"/>
         <!--box size="0.10 0.10 0.25"/-->
       </geometry>
@@ -17,5 +17,5 @@
       <origin xyz="0 0 0"/>
       <geometry>
-        <cylinder radius="0.01" length="0.08"/>
+        <cylinder radius="0.02" length="0.08"/>
         <!--box size="0.10 0.10 0.25"/-->
       </geometry>
