Commit message: feat: realize basic functions
Issue: shelf position and shape

File: kuka_arm/urdf/target.urdf.xacro (robot description, xacro)
@@ -10,5 +10,5 @@
       <origin xyz="0 0 0"/>
       <geometry>
-        <cylinder radius="0.02" length="0.08"/>
+        <cylinder radius="0.015" length="0.08"/>
         <!--box size="0.10 0.10 0.25"/-->
       </geometry>
@@ -17,5 +17,5 @@
       <origin xyz="0 0 0"/>
       <geometry>
-        <cylinder radius="0.02" length="0.08"/>
+        <cylinder radius="0.015" length="0.08"/>
         <!--box size="0.10 0.10 0.25"/-->
       </geometry>
