Commit message: feat: resolve target position problem
Issue: shelf rebuilding, gripper friction

File: kuka_arm/urdf/iiwa.gazebo.xacro (robot description, xacro)
@@ -22,5 +22,5 @@
     <!-- Link2 -->
     <gazebo reference="link_2">
-      <material>Gazebo/Orange</material>
+      <material>Gazebo/Grey</material>
       <mu1>0.2</mu1>
       <mu2>0.2</mu2>
@@ -34,5 +34,5 @@
     <!-- Link4 -->
     <gazebo reference="link_4">
-      <material>Gazebo/Orange</material>
+      <material>Gazebo/Grey</material>
       <mu1>0.2</mu1>
       <mu2>0.2</mu2>
@@ -46,5 +46,5 @@
     <!-- Link6 -->
     <gazebo reference="link_6">
-      <material>Gazebo/Orange</material>
+      <material>Gazebo/Grey</material>
       <mu1>0.2</mu1>
       <mu2>0.2</mu2>

File: kuka_arm/urdf/iiwa14.xacro (robot description, xacro)
@@ -35,5 +35,5 @@
         <origin xyz="-0.1 0 0.07" rpy="0 0 0"/>
         <mass value="50"/>
-        <inertia ixx="0.5"  ixy="0"  ixz="0" iyy="0.6" iyz="0" izz="0.3" />
+        <inertia ixx="5"  ixy="0"  ixz="0" iyy="6" iyz="0" izz="3" />
       </inertial>
       <visual>

File: kuka_arm/urdf/iiwa_gripper.xacro (robot description, xacro)
@@ -74,5 +74,5 @@
     <child link="right_gripper_finger_link" />
     <axis xyz="0 1 0" />
-    <limit effort="100" lower="-0.01" upper="${0.06/2}" velocity="0.05" />
+    <limit effort="100" lower="-0.01" upper="0.03" velocity="0.5" />
     <dynamics damping="0.7" friction="1.0"/>
   </joint>
@@ -82,5 +82,5 @@
     <child link="left_gripper_finger_link" />
     <axis xyz="0 -1 0" />
-    <limit effort="100" lower="-0.01" upper="${0.06/2}" velocity="0.05" />
+    <limit effort="100" lower="-0.01" upper="0.03" velocity="0.5" />
     <dynamics damping="0.7" friction="1.0"/>
   </joint>

File: kuka_arm/urdf/target.urdf.xacro (robot description, xacro)
@@ -5,5 +5,5 @@
       <origin xyz="0 0 0" />
       <mass value="0.1" />
-      <inertia  ixx="0.006" ixy="0"  ixz="0"  iyy="0.006"  iyz="0"  izz="0.002"/>
+      <inertia  ixx="0.00006" ixy="0"  ixz="0"  iyy="0.00006"  iyz="0"  izz="0.00002"/>
     </inertial>
     <visual>
