Commit message: feat: add gripper

File: iiwa_arm/urdf/iiwa14.urdf.xacro (robot description, xacro)
@@ -5,10 +5,12 @@
   <!--Import the lbr iiwa macro -->
   <xacro:include filename="$(find iiwa_arm)/urdf/iiwa14.xacro"/>
+  <!--Import the gripper macro -->
+  <xacro:include filename="$(find iiwa_arm)/urdf/iiwa_gripper.xacro"/>
+  <!--<xacro:include filename="$(find slam_project)/urdf/accessories/hexagons.urdf.xacro"/>-->
   <xacro:arg name="hardware_interface" default="PositionJointInterface"/>
   <xacro:arg name="robot_name" default="iiwa"/>
   <xacro:arg name="origin_xyz" default="0 0 0"/>
   <xacro:arg name="origin_rpy" default="0 0 0"/>
-  <!-- Fix to world just for testing -->
-  <!--<link name="world"/>-->
+  <!-- Fix to base_world -->
   <link name="base_footprint"/>
   <!--iiwa-->
@@ -16,3 +18,6 @@
     <origin xyz="$(arg origin_xyz)" rpy="$(arg origin_rpy)" />
   </xacro:iiwa14>
+  <!--gripper-->
+  <xacro:component_gripper robot_name="$(arg robot_name)" parent="$(arg robot_name)_link_ee">
+  </xacro:component_gripper>
 </robot>

File: iiwa_arm/urdf/iiwa14.xacro (robot description, xacro)
@@ -31,5 +31,5 @@
           <mesh filename="package://iiwa_arm/meshes/iiwa14/visual/link_0.stl"/>
         </geometry>
-        <material name="Grey"/>
+        <material name="LightGrey"/>
       </visual>
       <collision>
@@ -38,5 +38,5 @@
           <mesh filename="package://iiwa_arm/meshes/iiwa14/collision/link_0.stl"/>
         </geometry>
-        <material name="Grey"/>
+        <material name="LightGrey"/>
       </collision>
       <self_collision_checking>
@@ -107,5 +107,5 @@
           <mesh filename="package://iiwa_arm/meshes/iiwa14/visual/link_2.stl"/>
         </geometry>
-        <material name="Orange"/>
+        <material name="LightGrey"/>
       </visual>
       <collision>
@@ -114,5 +114,5 @@
           <mesh filename="package://iiwa_arm/meshes/iiwa14/collision/link_2.stl"/>
         </geometry>
-        <material name="Orange"/>
+        <material name="LightGrey"/>
       </collision>
     </link>
@@ -177,5 +177,5 @@
           <mesh filename="package://iiwa_arm/meshes/iiwa14/visual/link_4.stl"/>
         </geometry>
-        <material name="Orange"/>
+        <material name="LightGrey"/>
       </visual>
       <collision>
@@ -184,5 +184,5 @@
           <mesh filename="package://iiwa_arm/meshes/iiwa14/collision/link_4.stl"/>
         </geometry>
-        <material name="Orange"/>
+        <material name="LightGrey"/>
       </collision>
     </link>
@@ -247,5 +247,5 @@
           <mesh filename="package://iiwa_arm/meshes/iiwa14/visual/link_6.stl"/>
         </geometry>
-        <material name="Orange"/>
+        <material name="LightGrey"/>
       </visual>
       <collision>
@@ -254,5 +254,5 @@
           <mesh filename="package://iiwa_arm/meshes/iiwa14/collision/link_6.stl"/>
         </geometry>
-        <material name="Orange"/>
+        <material name="LightGrey"/>
       </collision>
     </link>

File: iiwa_arm/urdf/materials.xacro (robot description, xacro)
@@ -13,4 +13,7 @@
     <color rgba="0.4 0.4 0.4 1.0"/>
   </material>
+  <material name="LightGrey">
+    <color rgba="0.5 0.5 0.5 1.0"/>
+  </material>
   <material name="Orange">
     <color rgba="${255/255} ${108/255} ${10/255} 1.0"/>

Commit message: feat: revise controller association for moveit
Issue: src doesn't work correctly.

File: iiwa_arm/urdf/iiwa14.urdf.xacro (robot description, xacro)
@@ -19,5 +19,5 @@
   </xacro:iiwa14>
   <!--gripper-->
-  <xacro:component_gripper robot_name="$(arg robot_name)" parent="$(arg robot_name)_link_ee">
+  <xacro:component_gripper robot_name="$(arg robot_name)" parent="$(arg robot_name)_link_7">
   </xacro:component_gripper>
 </robot>

File: iiwa_arm/urdf/iiwa14.xacro (robot description, xacro)
@@ -292,5 +292,5 @@
       </collision>
     </link>
-    <joint name="${robot_name}_joint_ee" type="fixed">
+    <!--<joint name="${robot_name}_joint_ee" type="fixed">
       <parent link="${robot_name}_link_7"/>
       <child link="${robot_name}_link_ee"/>
@@ -298,5 +298,5 @@
     </joint>
     <link name="${robot_name}_link_ee">
-    </link>
+    </link>-->
     <!--Extensions -->
     <xacro:iiwa_gazebo robot_name="${robot_name}" />

File: iiwa_arm/urdf/iiwa_gripper.xacro (robot description, xacro)
@@ -3,5 +3,5 @@
   Hexagon stacks
  -->
-<robot name="component_gripper" xmlns:xacro="http://ros.org/wiki/xacro">
+<robot name="component_gripper" xmlns:xacro="http://www.ros.org/wiki/xacro">
   <xacro:property name="M_PI" value="3.1415926535897931" />
   <!-- Xacro properties -->
@@ -11,5 +11,5 @@
   <!-- Xacro macros -->
   <xacro:macro name="component_gripper" params="robot_name parent">
-     <link name="gripper_link">
+  <link name="gripper_link">
     <inertial>
       <origin xyz="0 0 0" rpy="0 0 0"/>
@@ -68,4 +68,5 @@
     </collision>
   </link>
+  <!--Joints-->
   <joint name="right_gripper_finger_joint" type="prismatic">
     <origin rpy="0 0 0" xyz="${0.15/2} ${-0.0725/2.5} 0" />
@@ -87,7 +88,8 @@
     <parent link="${parent}"/>
     <child link="gripper_link"/>
-    <origin xyz="0 0 0.035" rpy="0 -${M_PI/2} 0"/>
+    <origin xyz="0 0 ${0.045+0.035}" rpy="0 -${M_PI/2} 0"/>
     <axis xyz="0 1 0" />
   </joint>
+<!--transmissions-->
   <transmission name="${robot_name}_tran8">
     <type>transmission_interface/SimpleTransmission</type>

Commit message: chore: add world link into urdf

File: iiwa_arm/urdf/iiwa14.urdf.xacro (robot description, xacro)
@@ -12,6 +12,8 @@
   <xacro:arg name="origin_xyz" default="0 0 0"/>
   <xacro:arg name="origin_rpy" default="0 0 0"/>
+  <!-- Fix to world just for testing -->
+  <link name="world"/>
   <!--iiwa-->
-  <xacro:iiwa14 hardware_interface="$(arg hardware_interface)" robot_name="$(arg robot_name)">
+  <xacro:iiwa14 hardware_interface="$(arg hardware_interface)" robot_name="$(arg robot_name)" parent="world">
     <origin xyz="$(arg origin_xyz)" rpy="$(arg origin_rpy)" />
   </xacro:iiwa14>

File: iiwa_arm/urdf/iiwa14.xacro (robot description, xacro)
@@ -13,11 +13,11 @@
   <xacro:property name="max_effort" value="300"/>
   <xacro:property name="max_velocity" value="10"/>
-  <xacro:macro name="iiwa14" params="hardware_interface robot_name *origin">
+  <xacro:macro name="iiwa14" params="parent hardware_interface robot_name *origin">
     <!--joint between {parent} and link_0-->
-    <!--<joint name="${parent}_${robot_name}_joint" type="fixed">
+    <joint name="${parent}" type="fixed">
       <xacro:insert_block name="origin"/>
       <parent link="${parent}"/>
-      <child link="${robot_name}_link_0"/>
-    </joint>-->
+      <child link="base_footprint"/>
+    </joint>
     <link name="base_footprint"/>
     <joint name="fixed_base_joint" type="fixed">

File: iiwa_arm/urdf/iiwa_gripper.xacro (robot description, xacro)
@@ -22,4 +22,5 @@
         <mesh filename="package://iiwa_arm/meshes/gripper/gripper_base.dae" scale="0.5 0.4 0.3"/>
       </geometry>
+      <material name="LightGrey"/>
     </visual>
     <collision>
@@ -41,4 +42,5 @@
         <mesh filename="package://iiwa_arm/meshes/gripper/finger_right.dae" scale="0.5 0.5 0.5"/>
       </geometry>
+      <material name="LightGrey"/>
     </visual>
     <collision>
@@ -60,4 +62,5 @@
         <mesh filename="package://iiwa_arm/meshes/gripper/finger_left.dae" scale="0.5 0.5 0.5"/>
       </geometry>
+      <material name="LightGrey"/>
     </visual>
     <collision>
@@ -75,5 +78,5 @@
     <axis xyz="0 1 0" />
     <limit effort="100" lower="-0.01" upper="0.03" velocity="0.5" />
-    <dynamics damping="0.7" friction="0.5"/>
+    <dynamics damping="0.5"/>
   </joint>
   <joint name="left_gripper_finger_joint" type="prismatic">
@@ -83,5 +86,5 @@
     <axis xyz="0 -1 0" />
     <limit effort="100" lower="-0.01" upper="0.03" velocity="0.5" />
-    <dynamics damping="0.7" friction="0.5"/>
+    <dynamics damping="0.5"/>
   </joint>
   <joint name="gripper_joint" type="fixed">
@@ -130,4 +133,23 @@
     </plugin>
   </gazebo>
+  <!--material-->
+  <!-- gripper_link -->
+  <gazebo reference="gripper_link">
+    <material>Gazebo/Grey</material>
+    <mu1>0.2</mu1>
+    <mu2>0.2</mu2>
+  </gazebo>
+  <!-- left_gripper_finger_link -->
+  <gazebo reference="left_gripper_finger_link">
+    <material>Gazebo/Grey</material>
+    <mu1>1.0</mu1>
+    <mu2>1.0</mu2>
+  </gazebo>
+  <!-- right_gripper_finger_link -->
+  <gazebo reference="right_gripper_finger_link">
+    <material>Gazebo/Grey</material>
+    <mu1>1.0</mu1>
+    <mu2>1.0</mu2>
+  </gazebo>
   </xacro:macro>
 </robot>
