Commit message: feat: implement basic IK
complex value problem

File: iiwa_arm/urdf/iiwa14.xacro (robot description, xacro)
@@ -134,5 +134,7 @@
       <origin xyz="0 0.2045 0" rpy="${PI / 2} 0 ${PI}"/>
       <axis xyz="0 0 1"/>
-      <limit lower="${-170 * PI / 180}" upper="${170 * PI / 180}"
+      <!--<limit lower="${-170 * PI / 180}" upper="${170 * PI / 180}"
+             effort="${max_effort}" velocity="${max_velocity}" />-->
+      <limit lower="${0}" upper="${0}"
              effort="${max_effort}" velocity="${max_velocity}" />
       <safety_controller soft_lower_limit="${-168 * PI / 180}"

File: iiwa_arm/urdf/iiwa_gripper.xacro (robot description, xacro)
@@ -92,4 +92,5 @@
     <child link="gripper_link"/>
     <origin xyz="0 0 ${0.045+0.035}" rpy="0 -${M_PI/2} 0"/>
+    <!--<origin xyz="0 0 ${0.045+0.035}" rpy="0 0 0"/>-->
     <axis xyz="0 1 0" />
   </joint>

Commit message: feat: IK works!
Issue:  arm lagging

File: iiwa_arm/urdf/iiwa14.xacro (robot description, xacro)
@@ -134,8 +134,8 @@
       <origin xyz="0 0.2045 0" rpy="${PI / 2} 0 ${PI}"/>
       <axis xyz="0 0 1"/>
-      <!--<limit lower="${-170 * PI / 180}" upper="${170 * PI / 180}"
+      <limit lower="${-170 * PI / 180}" upper="${170 * PI / 180}"
+             effort="${max_effort}" velocity="${max_velocity}" />
+      <!--<limit lower="${0}" upper="${0}"
              effort="${max_effort}" velocity="${max_velocity}" />-->
-      <limit lower="${0}" upper="${0}"
-             effort="${max_effort}" velocity="${max_velocity}" />
       <safety_controller soft_lower_limit="${-168 * PI / 180}"
                          soft_upper_limit="${168 * PI / 180}"

Commit message: feat: rebuild movit! files

File: iiwa_arm/urdf/iiwa14.xacro (robot description, xacro)
@@ -27,14 +27,14 @@
     </joint>
     <link name="base_link">
-      <!--<inertial>
+      <inertial>
         <origin xyz="-0.1 0 0.07" rpy="0 0 0"/>
         <mass value="5"/>
         <inertia ixx="0.05"  ixy="0"  ixz="0" iyy="0.06" iyz="0" izz="0.03" />
-      </inertial>-->
-      <inertial>
+      </inertial>
+      <!--<inertial>
         <origin xyz="-0.1 0 0.07" rpy="0 0 0"/>
         <mass value="50"/>
         <inertia ixx="5"  ixy="0"  ixz="0" iyy="6" iyz="0" izz="3" />
-      </inertial>
+      </inertial>-->
       <visual>
         <origin xyz="0 0 0" rpy="0 0 0"/>
